File: KiCad Stuff/half-life-starbieee.kicad_sch (KiCad schematic)
At the start: 0 parts

Commit message: kicad works
Parts:
- added J1: Conn_01x04_Pin, symbol Connector:Conn_01x04_Pin
- added J2: Conn_01x08_Pin, Package_DIP:DIP-20_W7.62mm, symbol Connector:Conn_01x08_Pin
- added R1: 10k, Package_DIP:DIP-8_W7.62mm, symbol Device:R
- added SW1: SW_Push, Package_DIP:DIP-8_W7.62mm, symbol Switch:SW_Push
- added SW2: SW_Push, symbol Switch:SW_Push
- added U1: XIAO-ESP32-C3-SMD, Seeed_Studio_XIAO_Series:XIAO-ESP32-C3-SMD, symbol symbols:XIAO-ESP32-C3-SMD
- added U2: DHT11, Sensor:Aosong_DHT11_5.5x12.0_P2.54mm, symbol Sensor:DHT11
Connections:
- new net +3.3V: J1.2 (Pin_2), J2.1 (Pin_1), R1.2, U1.12 (3V3_OUT), U2.1 (VDD)
- new net +5V: U1.14 (VBUS)
- new net B_1: SW1.1, U1.3 (D2)
- new net B_2: SW2.1, U1.4 (D3)
- new net DHT11_DAT: R1.1, U1.2 (D1), U2.2 (DATA)
- new net GND: J1.1 (Pin_1), J2.2 (Pin_2), SW1.2, SW2.2, U1.13 (GND), U1.18 (GND), U2.4 (GND)
- new net SCL: J1.3 (Pin_3), J2.3 (Pin_3), U1.5 (D4)
- new net SDA: J1.4 (Pin_4), J2.4 (Pin_4), U1.6 (D5)
- no-connect marks 0 -> 17

Commit message: kicad works
Parts:
- added SW3: RotaryEncoder_Switch_MP, Rotary_Encoder:RotaryEncoder_Alps_EC11E-Switch_Vertical_H20mm, symbol Device:RotaryEncoder_Switch_MP
- J1: footprint (none) -> Imported Parts:Display_128x64_096_I2C
- J2: footprint Package_DIP:DIP-20_W7.62mm -> Connector_PinHeader_2.00mm:PinHeader_1x08_P2.00mm_Vertical
- R1: footprint Package_DIP:DIP-8_W7.62mm -> Resistor_SMD:R_0805_2012Metric
- SW1: footprint Package_DIP:DIP-8_W7.62mm -> Button_Switch_Keyboard:SW_Cherry_MX_1.00u_PCB
- SW2: footprint (none) -> Button_Switch_Keyboard:SW_Cherry_MX_1.00u_PCB
- U1: footprint Seeed_Studio_XIAO_Series:XIAO-ESP32-C3-SMD -> Imported Parts:XIAO-ESP32-C6-DIP
Connections:
- net GND: now also SW3.C, SW3.MP, SW3.S2
- net RE1_B: now reaches U1.8 (D7)
- net RE1_B: now also SW3.B
- net RE1_A: now reaches U1.9 (D8)
- net RE1_A: now also SW3.A
- net B_1 renamed B1
- net B_2 renamed B2
- new net RE_B3: SW3.S1
- no-connect marks 17 -> 15
