File: kicad/half-life-starbieee.kicad_sch (KiCad schematic)
At the start: 8 parts, among them J1 Conn_01x04_Pin, J2 Conn_01x08_Pin, SW1 SW_Push, SW2 SW_Push, SW3 RotaryEncoder_Switch_MP, U1 XIAO-ESP32-C3-SMD, U2 DHT11

Commit message: readme + arduino stuff
Connections:
- net RE_B3: now also U1.11 (D10)
- no-connect marks 15 -> 14
Changed lines of the file:
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@@
-	)
-	(no_connect
-		(at 67.31 45.72)
 	)
 	(no_connect
@@
 		(pts
 			(xy 93.98 26.67) (xy 90.17 26.67)
+		)
+		(stroke
+			(width 0)
+			(type default)
+		)
+	)
+	(wire
+		(pts
+			(xy 67.31 45.72) (xy 74.93 45.72)
 		)
 		(stroke
@@
 		)
 	)
+	(label "RE_B3"
+		(at 74.93 45.72 180)
+		(effects
+			(font
+				(size 1.27 1.27)
+			)
+			(justify right bottom)
+		)
+	)
